File: Hardware/Bus_switch.kicad_sch (KiCad schematic)
At the start: 15 parts, among them J3 Conn_01x04_Pin, U1 SN74CB3Q3384APW

Commit message: made pcb
Parts:
- removed J3: Conn_01x04_Pin, Connector_PinHeader_2.54mm:PinHeader_1x04_P2.54mm_Vertical, symbol Connector:Conn_01x04_Pin
- removed R1: 330Ω, PCM_JLCPCB:R_0402, symbol PCM_JLCPCB-Resistors:0402,330Ω
- removed R10, R11, R2, R3, R4, R5, R6, R7, R8, R9: 10kΩ, PCM_JLCPCB:R_0402, symbol PCM_JLCPCB-Resistors:0402,10kΩ
- added R1, R2, R3, R4, R6, R8, R9: 10kΩ, PCM_JLCPCB:R_0603, symbol PCM_JLCPCB-Resistors:0603,10kΩ
- added R7: 1kΩ, PCM_JLCPCB:R_0603, symbol PCM_JLCPCB-Resistors:0603,1kΩ
Connections:
- net +3V3: now also R2.1, R3.1, R4.1, R6.1, R9.1
- net Chainbus.CS: now also R3.2
- net Chainbus.MOSI: now also R1.1
- net Chainbus.SCK: now also R2.2, R8.1
- net Chainbus.SCL: now also R9.2
- net Chainbus.SDA: now also R6.2
- net GND: now also R1.2, R8.2
- net SEL1: now also R4.2, R7.1
- net at D3.1: now also R7.2
Other:
- note added: "We don't have standard EEPROM"
- company: (none) -> MiniModucard System
- title: MMS3 Hat template small (Change Me) -> MMS3 Hat Hat Expander
