File: Hardware/MMS3_hat_templates.kicad_pcb (KiCad board)
At the start: 2 copper layers, 100 x 50 mm, 28 parts, among them J1 Chainbus in, J2 Chainbus Out, J3 Conn_01x04_Pin, J4 AMASS XT60 Male, J5 AMASS XT60 Female, U1 SN74CB3Q3384APW, U2 M24C64, U4 AMS1117

Commit message: made pcb
Parts:
- removed C2: 100nF, PCM_JLCPCB:C_0603
- removed D1: M7, PCM_JLCPCB:D_SMA
- removed J3: Conn_01x04_Pin, Connector_PinHeader_2.54mm:PinHeader_1x04_P2.54mm_Vertical
- removed J4: AMASS XT60 Male, XT60:AMASS_XT60PW-M_1x02_P7.20mm_Horizontal
- removed U2: M24C64, PCM_JLCPCB:SOIC-8_L5.0-W4.0-P1.27-LS6.0-BL
- added C3: 100nF, PCM_JLCPCB:C_0603, F.Cu at (158.6, 97.9)
- added C4: 12pF, PCM_JLCPCB:C_0603, F.Cu at (162.5, 95.3)
- added C5: 12pF, PCM_JLCPCB:C_0603, F.Cu at (157.8, 95.2)
- added D10: Red, PCM_JLCPCB:D_0603, F.Cu at (121.7, 131.5)
- added D11: Red, PCM_JLCPCB:D_0603, F.Cu at (127.8, 131.5)
- added D12: Red, PCM_JLCPCB:D_0603, F.Cu at (129.8, 131.5)
- added D13: Red, PCM_JLCPCB:D_0603, F.Cu at (131.8, 131.5)
- added D14: Red, PCM_JLCPCB:D_0603, F.Cu at (133.8, 131.5)
- added D15: Red, PCM_JLCPCB:D_0603, F.Cu at (135.8, 131.5)
- added D16: Red, PCM_JLCPCB:D_0603, F.Cu at (137.8, 131.5)
- added D17: Red, PCM_JLCPCB:D_0603, F.Cu at (139.8, 131.5)
- added D18: Red, PCM_JLCPCB:D_0603, F.Cu at (141.8, 131.5)
- added D2: Red, PCM_JLCPCB:D_0603, F.Cu at (107.7, 131.5)
- added D4: Red, PCM_JLCPCB:D_0603, F.Cu at (109.7, 131.5)
- added D5: Red, PCM_JLCPCB:D_0603, F.Cu at (111.7, 131.5)
- added D6: Red, PCM_JLCPCB:D_0603, F.Cu at (113.7, 131.5)
- added D7: Red, PCM_JLCPCB:D_0603, F.Cu at (115.7, 131.5)
- added D8: Red, PCM_JLCPCB:D_0603, F.Cu at (117.7, 131.5)
- added D9: Red, PCM_JLCPCB:D_0603, F.Cu at (119.7, 131.5)
- added R12: 1kΩ, PCM_JLCPCB:R_0603, F.Cu at (107.7, 128.5)
- added R15: 1kΩ, PCM_JLCPCB:R_0603, F.Cu at (109.7, 128.5)
- added R16: 1kΩ, PCM_JLCPCB:R_0603, F.Cu at (111.7, 128.5)
- added R17: 1kΩ, PCM_JLCPCB:R_0603, F.Cu at (113.7, 128.5)
- added R18: 1kΩ, PCM_JLCPCB:R_0603, F.Cu at (115.7, 128.5)
- added R19: 1kΩ, PCM_JLCPCB:R_0603, F.Cu at (117.7, 128.5)
- added R2: 10kΩ, PCM_JLCPCB:R_0603, F.Cu at (154.7, 101.0)
- added R20: 1kΩ, PCM_JLCPCB:R_0603, F.Cu at (119.7, 128.5)
- added R21: 1kΩ, PCM_JLCPCB:R_0603, F.Cu at (121.7, 128.5)
- added R22: 1kΩ, PCM_JLCPCB:R_0603, F.Cu at (127.8, 128.5)
- added R23: 1kΩ, PCM_JLCPCB:R_0603, F.Cu at (129.8, 128.5)
- added R24: 1kΩ, PCM_JLCPCB:R_0603, F.Cu at (131.8, 128.5)
- added R25: 1kΩ, PCM_JLCPCB:R_0603, F.Cu at (133.8, 128.5)
- added R26: 1kΩ, PCM_JLCPCB:R_0603, F.Cu at (135.8, 128.5)
- added R27: 1kΩ, PCM_JLCPCB:R_0603, F.Cu at (137.8, 128.5)
- added R28: 1kΩ, PCM_JLCPCB:R_0603, F.Cu at (139.8, 128.5)
- added R29: 1kΩ, PCM_JLCPCB:R_0603, F.Cu at (141.8, 128.5)
- added R3: 10kΩ, PCM_JLCPCB:R_0603, F.Cu at (155.9, 108.8)
- added R7: 1kΩ, PCM_JLCPCB:R_0603, F.Cu at (173.1, 98.0)
- added R8: 10kΩ, PCM_JLCPCB:R_0603, F.Cu at (152.7, 101.0)
- added R9: 10kΩ, PCM_JLCPCB:R_0603, F.Cu at (151.6, 106.0)
- added S1: Tactile Button, 160gf, PCM_JLCPCB:SW_TS-1088-AR02016, F.Cu at (173.7, 102.3)
- added U3: CH32V003FxPx, PCM_JLCPCB:TSSOP-20_4.4x6.5mm_P0.65mm, F.Cu at (160.5, 102.6)
- added X1: X322525MOB4SI, PCM_JLCPCB:OSC-SMD_4P-L3.2-W2.5-BL, F.Cu at (160.3, 95.2)
- J5: value AMASS XT60 Female -> Program; footprint XT60:AMASS_XT60PW-F_1x02_P7.20mm_Horizontal -> Connector_PinHeader_2.54mm:PinHeader_1x03_P2.54mm_Vertical
- R1: value 330Ω -> 10kΩ; footprint PCM_JLCPCB:R_0402 -> PCM_JLCPCB:R_0603
- R10, R4, R6: footprint PCM_JLCPCB:R_0402 -> PCM_JLCPCB:R_0603
- moved C16 69.8 mm to (96.8, 94.6)
- moved C18 69.8 mm to (96.9, 96.9)
- moved U4 69.8 mm to (91.0, 96.9)
- moved J5 59.7 mm to (163.6, 108.9), turned to -90 degrees
- moved G*** 29.7 mm to (172.5, 98.8)
- moved R1 23.2 mm to (150.7, 101.0), turned to 90 degrees
- moved R10 18.4 mm to (168.8, 102.1), turned to 90 degrees
- moved R4 6.38 mm to (156.2, 99.0), turned to -90 degrees
- moved R6 1.41 mm to (153.0, 106.0), turned to -90 degrees
Connections:
- net /Bus_switch/Chainbus.MISO renamed /Chainbus.MISO
- net /Bus_switch/Chainbus_In.CS renamed /Chainbus_In.CS
- net /Bus_switch/Chainbus_In.MISO renamed /Chainbus_In.MISO
- net /Bus_switch/Chainbus_In.MOSI renamed /Chainbus_In.MOSI
- net /Bus_switch/Chainbus_In.RX renamed /Chainbus_In.RX
- net /Bus_switch/Chainbus_In.SCK renamed /Chainbus_In.SCK
- net /Bus_switch/Chainbus_In.SCL renamed /Chainbus_In.SCL
- net /Bus_switch/Chainbus_In.SDA renamed /Chainbus_In.SDA
- net /Bus_switch/Chainbus_In.TX renamed /Chainbus_In.TX
- J1 pad 10: /Interboard_connector/SEL5 -> /SEL_5
- J1 pad 12: /Interboard_connector/SEL6 -> /SEL_6
- J1 pad 14: /Interboard_connector/SEL7 -> /SEL_7
- J1 pad 16: /Interboard_connector/SEL8 -> /SEL_8
- J1 pad 2: /Bus_switch/SEL1 -> /SEL_1
- J1 pad 4: /Interboard_connector/SEL2 -> /SEL_2
- J1 pad 6: /Interboard_connector/SEL3 -> /SEL_3
- J1 pad 8: /Interboard_connector/SEL4 -> /SEL_4
- J2 pad 10: /Interboard_connector/SEL6 -> /NEW_SEL5
- J2 pad 12: /Interboard_connector/SEL7 -> /NEW_SEL6
- J2 pad 14: /Interboard_connector/SEL8 -> /NEW_SEL7
- J2 pad 16: unconnected-(J2-Pin_16-Pad16) -> /NEW_SEL8
- J2 pad 2: /Interboard_connector/SEL2 -> /NEW_SEL1
- J2 pad 4: /Interboard_connector/SEL3 -> /NEW_SEL2
- J2 pad 6: /Interboard_connector/SEL4 -> /NEW_SEL3
- J2 pad 8: /Interboard_connector/SEL5 -> /NEW_SEL4
- J5 pad 1: GND -> /CH32V003/SWIO
- J5 pad 2: /Power Connector/VIN_BRD -> GND
- R1 pad 1: /Bus_switch/SEL1 -> /Chainbus.MOSI
- R1 pad 2: Net-(D3-Pad1) -> GND
- R10 pad 2: /Bus_switch/Chainbus.SDA -> /CH32V003/PD7
- R4 pad 1: /Bus_switch/SEL1 -> +3V3
- R4 pad 2: +3V3 -> /SEL_1
- R6 pad 2: /Bus_switch/Chainbus.SCL -> /Chainbus.SDA
- U1 pad 1: /Bus_switch/SEL1 -> /SEL_1
- U1 pad 10: /Bus_switch/Chainbus.SCK -> /Chainbus.SCK
- U1 pad 13: /Bus_switch/SEL1 -> /SEL_1
- U1 pad 15: /Bus_switch/Chainbus.CS -> /Chainbus.CS
- U1 pad 16: /Bus_switch/Chainbus.SDA -> /Chainbus.SDA
- U1 pad 19: /Bus_switch/Chainbus.SCL -> /Chainbus.SCL
- U1 pad 9: /Bus_switch/Chainbus.MOSI -> /Chainbus.MOSI
Routing:
- net /SEL_1: track 0.00 -> 130.2 mm, vias 0 -> 7
- net +3V3: track 59.0 -> 179.9 mm, vias 4 -> 6
- net /NEW_SEL1: track 0.00 -> 93.8 mm, vias 0 -> 3
- net /NEW_SEL2: track 0.00 -> 90.6 mm, vias 0 -> 3
- net /NEW_SEL3: track 0.00 -> 87.9 mm, vias 0 -> 3
- net /NEW_SEL4: track 0.00 -> 87.5 mm, vias 0 -> 3
- net /Bus_switch/SEL1: track 82.8 -> 0.00 mm, vias 4 -> 0
- net /NEW_SEL5: track 0.00 -> 74.4 mm, vias 0 -> 3
- net /NEW_SEL6: track 0.00 -> 69.3 mm, vias 0 -> 3
- net /NEW_SEL7: track 0.00 -> 65.6 mm, vias 0 -> 3
- net /NEW_SEL8: track 0.00 -> 64.8 mm, vias 0 -> 3
- net /SEL_8: track 0.00 -> 41.1 mm, vias 0 -> 1
- net /SEL_7: track 0.00 -> 40.7 mm, vias 0 -> 1
- net /SEL_6: track 0.00 -> 40.6 mm, vias 0 -> 1
- net /SEL_5: track 0.00 -> 40.3 mm, vias 0 -> 1
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- removed copper zone on F.Cu, net /Power Connector/VIN_BRD
Other:
- board text added: "CH32v003"
- board text added: "Input"
- board text added: "MMS3 Hat Hat-Hat expander Version 1.0 Made By Wojeciech Sz."
- board text added: "Output"
- board text added: "RESET"
- board text added: "SEL1"
- board text added: "SEL2"
- board text added: "SEL3"
- board text added: "SEL4"
- board text added: "SEL5"
- board text added: "SEL6"
- board text added: "SEL7"
- board text added: "SEL8"
- board text added: "SWIO"
- board text removed: "SCL"
- board text removed: "SDA"
