File: Hardware/MMS3_hat_templates.kicad_sch (KiCad schematic)
At the start: 12 parts, among them U4 AMS1117

Commit message: made pcb
Parts:
- added D10, D11, D12, D13, D14, D15, D16, D17, D18, D2, D4, D5, D6, D7, D8, D9: Red, PCM_JLCPCB:D_0603, symbol PCM_JLCPCB-Diodes:LED,0603,Red
- added J1: Chainbus in, Connector_PinHeader_2.54mm:PinHeader_2x16_P2.54mm_Vertical_SMD, symbol Connector_Generic:Conn_02x16_Odd_Even
- added J2: Chainbus Out, Connector_PinSocket_2.54mm:PinSocket_2x16_P2.54mm_Vertical_SMD, symbol Connector_Generic:Conn_02x16_Odd_Even
- added R12, R15, R16, R17, R18, R19, R20, R21, R22, R23, R24, R25, R26, R27, R28, R29: 1kΩ, PCM_JLCPCB:R_0603, symbol PCM_JLCPCB-Resistors:0603,1kΩ
Connections:
- net +3V3: now also D10.2, D11.2, D12.2, D13.2, D14.2, D15.2, D16.2, D17.2, D18.2, D2.2, D4.2, D5.2, D6.2, D7.2, D8.2, D9.2
- net +5V: now also J1.3 (Pin_3), J1.5 (Pin_5), J2.3 (Pin_3), J2.5 (Pin_5)
- net GND: now also J1.1 (Pin_1), J1.17 (Pin_17), J1.19 (Pin_19), J1.21 (Pin_21), J1.23 (Pin_23), J1.31 (Pin_31), J1.7 (Pin_7), J2.1 (Pin_1), J2.17 (Pin_17), J2.19 (Pin_19), J2.21 (Pin_21), J2.23 (Pin_23), J2.31 (Pin_31), J2.7 (Pin_7)
- net VIN_CHAINBUS: now also J1.11 (Pin_11), J1.13 (Pin_13), J1.15 (Pin_15), J1.9 (Pin_9), J2.11 (Pin_11), J2.13 (Pin_13), J2.15 (Pin_15), J2.9 (Pin_9)
- new net: D2.1, R12.1
- new net: D13.1, R24.1
- new net: D10.1, R21.1
- new net: D5.1, R16.1
- new net: D7.1, R18.1
- new net: D17.1, R28.1
- new net: D16.1, R27.1
- new net: D4.1, R15.1
- new net: D12.1, R23.1
- new net: D15.1, R26.1
- new net: D6.1, R17.1
- new net: D9.1, R20.1
- new net: D18.1, R29.1
- new net: D8.1, R19.1
- new net: D14.1, R25.1
- new net: D11.1, R22.1
- new net +12V stby: J1.29 (Pin_29), J2.29 (Pin_29)
- new net Chainbus_In.CS: J1.22 (Pin_22), J2.22 (Pin_22)
- new net Chainbus_In.MISO: J1.28 (Pin_28), J2.28 (Pin_28)
- new net Chainbus_In.MOSI: J1.26 (Pin_26), J2.26 (Pin_26)
- new net Chainbus_In.RX: J1.32 (Pin_32), J2.32 (Pin_32)
- new net Chainbus_In.SCK: J1.24 (Pin_24), J2.24 (Pin_24)
- new net Chainbus_In.SCL: J1.20 (Pin_20), J2.20 (Pin_20)
- new net Chainbus_In.SDA: J1.18 (Pin_18), J2.18 (Pin_18)
- new net Chainbus_In.TX: J1.30 (Pin_30), J2.30 (Pin_30)
- new net NEW_SEL1: J2.2 (Pin_2), R22.2
- new net NEW_SEL2: J2.4 (Pin_4), R23.2
- new net NEW_SEL3: J2.6 (Pin_6), R24.2
- new net NEW_SEL4: J2.8 (Pin_8), R25.2
- new net NEW_SEL5: J2.10 (Pin_10), R26.2
- new net NEW_SEL6: J2.12 (Pin_12), R27.2
- new net NEW_SEL7: J2.14 (Pin_14), R28.2
- new net NEW_SEL8: J2.16 (Pin_16), R29.2
- new net SEL_1: J1.2 (Pin_2), R12.2
- new net SEL_2: J1.4 (Pin_4), R15.2
- new net SEL_3: J1.6 (Pin_6), R16.2
- new net SEL_4: J1.8 (Pin_8), R17.2
- new net SEL_5: J1.10 (Pin_10), R18.2
- new net SEL_6: J1.12 (Pin_12), R19.2
- new net SEL_7: J1.14 (Pin_14), R20.2
- new net SEL_8: J1.16 (Pin_16), R21.2
- no-connect marks 0 -> 9
Other:
- removed sheet ID EEPROM
- removed sheet Interboard_connector
- removed sheet Power Connector
- added sheet CH32V003 (CH32V003.kicad_sch)
- note added: "ChainBus In"
- note added: "ChainBus Out"
- note added: "Indicator LED's (ooo blinky)"
- note added: "This boy Right Here is our EEPROM"
- note removed: "<-- Use those connections"
- note removed: "Chainbus connector and bus switch - Do Not Modify"
- note removed: "ID"
- title: MMS3 Hat template small (Change Me) -> MMS3 Hat Hat Expander
